File: Clock_Input_SingleEnded_Out.kicad_sch (KiCad schematic)
At the start: 23 parts, among them IC12 THS4541IRGTT, J9 SMA, U10 LTC6752ISC6-4#TRMPBF

Commit message: Document A bit and add more silkscreen
Parts:
- IC12: footprint Package_DFN_QFN:VQFN-16-1EP_3x3mm_P0.5mm_EP1.45x1.45mm -> 1_Footprint_Library:VQFN-16-1EP_3x3mm_P0.5mm_EP1.45x1.45mm
Changed lines of the file:
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@@
 			)
 		)
-		(property "Footprint" "Package_DFN_QFN:VQFN-16-1EP_3x3mm_P0.5mm_EP1.45x1.45mm"
+		(property "Footprint" "1_Footprint_Library:VQFN-16-1EP_3x3mm_P0.5mm_EP1.45x1.45mm"
 			(at 138.43 136.906 0)
 			(effects
